File: portable_FM_DIP.brd (EAGLE design)
At the start: 31 parts, among them J1 LCD HD44780 8x2, J2 2x3 ICSP Male, J3 VIN From Lipo Rider, J4 Pololu Variable reg 3.3V Out

Commit message: Code and Updated Board
Routing:
- net S$5: track 46.9 -> 48.7 mm, vias 0 -> 1
- removed copper zone on layer 1, net GND
- removed copper zone on layer 16, net GND
Changed lines of the file:
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@@
 <setting verticaltext="up"/>
 </settings>
-<grid distance="1" unitdist="mm" unit="mm" style="lines" multiple="1" display="yes" altdistance="0.025" altunitdist="inch" altunit="inch"/>
+<grid distance="0.1" unitdist="mm" unit="mm" style="lines" multiple="1" display="yes" altdistance="0.025" altunitdist="inch" altunit="inch"/>
 <layers>
 <layer number="1" name="Top" color="4" fill="1" visible="yes" active="yes"/>
@@
 <wire x1="14.5" y1="33.9" x2="31.7" y2="33.9" width="0.4064" layer="1"/>
 <wire x1="31.7" y1="33.9" x2="35.1" y2="30.5" width="0.4064" layer="1"/>
-<wire x1="35.1" y1="30.5" x2="35.1" y2="22.6" width="0.4064" layer="1"/>
-<wire x1="35.1" y1="22.6" x2="29" y2="16.5" width="0.4064" layer="1"/>
-<wire x1="27.2" y1="16.5" x2="29" y2="16.5" width="0.4064" layer="1"/>
+<wire x1="35.1" y1="30.5" x2="35.1" y2="26.5" width="0.4064" layer="1"/>
 <wire x1="13.5" y1="29.2" x2="12.6" y2="29.2" width="0.4064" layer="1"/>
 <wire x1="12.6" y1="29.2" x2="12.4" y2="29.4" width="0.4064" layer="1"/>
 <wire x1="12.4" y1="29.4" x2="12.4" y2="31.8" width="0.4064" layer="1"/>
 <wire x1="12.4" y1="31.8" x2="14.5" y2="33.9" width="0.4064" layer="1"/>
+<via x="36.3" y="25.3" extent="1-16" drill="0.6" diameter="1.4224" shape="square"/>
+<wire x1="35.1" y1="26.5" x2="36.3" y2="25.3" width="0.4064" layer="1"/>
+<wire x1="36.3" y1="25.3" x2="36.3" y2="22.4" width="0.4064" layer="16"/>
+<wire x1="36.3" y1="22.4" x2="30.6" y2="16.7" width="0.4064" layer="16"/>
+<wire x1="27.2" y1="16.5" x2="30.4" y2="16.5" width="0.4064" layer="16"/>
+<wire x1="30.4" y1="16.5" x2="30.6" y2="16.7" width="0.4064" layer="16"/>
 </signal>
 <signal name="S$52">
@@
 <wire x1="29.7" y1="34.7" x2="30.4" y2="34" width="0.4064" layer="16"/>
 <wire x1="18.6" y1="43.6" x2="18.6" y2="47" width="0.4064" layer="1"/>
-<polygon width="0.4064" layer="1">
-<vertex x="2" y="76"/>
-<vertex x="56" y="76"/>
-<vertex x="56" y="2"/>
-<vertex x="2" y="2"/>
-</polygon>
-<polygon width="0.4064" layer="16">
-<vertex x="2" y="76"/>
-<vertex x="56" y="76"/>
-<vertex x="56" y="2"/>
-<vertex x="2" y="2"/>
-</polygon>
 <wire x1="28.7" y1="36.8" x2="28.7" y2="37.6" width="0" layer="19" extent="1-16"/>
 </signal>
